File: SiPM_Breakout/SiPM_Breakout.kicad_pcb (KiCad board)
At the start: 2 copper layers, 1 part, among them U1 MICROFC-60035-SMT-TR

Commit message: Finished Annotations + Completed PCB
Parts:
- added C1: 10 nF, Capacitor_SMD:C_0805_2012Metric_Pad1.18x1.45mm_HandSolder, F.Cu at (133.5, 99.0)
- added J1: K, Connector_PinHeader_1.00mm:PinHeader_1x01_P1.00mm_Vertical, F.Cu at (149.5, 89.5)
- added J2: F_Out, Connector_PinHeader_1.00mm:PinHeader_1x01_P1.00mm_Vertical, F.Cu at (149.5, 95.5)
- added J3: A, Connector_PinHeader_1.00mm:PinHeader_1x01_P1.00mm_Vertical, F.Cu at (132.5, 96.0)
- added J4: NC, Connector_PinHeader_1.00mm:PinHeader_1x01_P1.00mm_Vertical, F.Cu at (132.5, 89.5)
- U1: footprint MICROFC-60035-SMT-TR:ON_Semiconductor-512AG-07_2018-O-MFG -> Onsemi:ON_Semiconductor-512AG-07_2018-O-MFG
Connections:
- U1 pad 1: unconnected-(U1-Anode-Pad1) -> Net-(J3-Pin_1)
- U1 pad 2: unconnected-(U1-Fast_Output-Pad2) -> Net-(J2-Pin_1)
- U1 pad 3: unconnected-(U1-Cathode-Pad3) -> Net-(J1-Pin_1)
- U1 pad 4: unconnected-(U1-NC-Pad4) -> GNDREF
Routing:
- net Net-(J1-Pin_1): track 0.00 -> 21.3 mm, vias 0 -> 2
- net Net-(J3-Pin_1): track 0.00 -> 8.81 mm
- net GNDREF: track 0.00 -> 6.05 mm
- net Net-(J2-Pin_1): track 0.00 -> 5.50 mm
Other:
- board outline added: 22 x 15.5 mm
- board text added: "Muon Detector SiPM Breakout"
- board text added: "Tyler Roche, JuaN Fritschy, Bartol Barcot (Scintillator)"
